File: ServoLaser/ServoLaser.kicad_pcb (KiCad board)
At the start: 2 copper layers, 30.5 x 25.4 mm, 9 parts, among them J1 Conn_01x03, J2 Conn_01x03, J3 ICSP, U2 ATTINY85-20PU

Commit message: change name
Other:
- board text added: "Maniacal Labs ServoBuddy"
- board text removed: "Maniacal Labs ServoLaser"
